File: syzygy-breakout-flash-1V8XL.kicad_pcb (KiCad board)
At the start: 4 copper layers, 105.6 x 76 mm, 33 parts, among them J1 QTE-020-01-F-D-A-TR, J10 TagConnect, J11 Conn_01x08, J12 Conn_01x02, J13 Conn_01x02, J14 Conn_01x04, J15 Conn_01x08, J2 QTE-020-01-F-D-A-TR, J3 Conn_01x04, J4 Conn_01x03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

Commit message: feat(pcb): push latest verified pcb design
Parts:
- D1: moved to B.Cu
Changed lines of the file:
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@@
     )
   )
-  (footprint "Diode_SMD:D_SOD-323" (layer "F.Cu")
-    (at 185.17 75.1775 90)
-    (descr "SOD-323")
-    (tags "SOD-323")
-    (property "Sheetfile" "pdclk.kicad_sch")
-    (property "Sheetname" "PD and CLK")
-    (property "ki_description" "10V 3A High Current Recitifier Schottky Diode, SOD-323")
-    (property "ki_keywords" "diode Schottky")
-    (attr smd)
-    (fp_text reference "D1" (at 0 -1.85 90) (layer "F.SilkS")
-        (effects (font (size 1 1) (thickness 0.15)))
-    )
-    (fp_text value "BAT60A" (at 0.1 1.9 90) (layer "F.Fab") hide
-        (effects (font (size 1 1) (thickness 0.15)))
-    )
-    (fp_text user "${REFERENCE}" (at 0 -1.85 90) (layer "F.Fab")
-        (effects (font (size 1 1) (thickness 0.15)))
-    )
-    (fp_line (start -1.61 -0.85) (end -1.61 0.85)
-      (stroke (width 0.12) (type solid)) (layer "F.SilkS"))
-    (fp_line (start -1.61 -0.85) (end 1.05 -0.85)
-      (stroke (width 0.12) (type solid)) (layer "F.SilkS"))
-    (fp_line (start -1.61 0.85) (end 1.05 0.85)
-      (stroke (width 0.12) (type solid)) (layer "F.SilkS"))
-    (fp_line (start -1.6 -0.95) (end -1.6 0.95)
-      (stroke (width 0.05) (type solid)) (layer "F.CrtYd"))
-    (fp_line (start -1.6 -0.95) (end 1.6 -0.95)
-      (stroke (width 0.05) (type solid)) (layer "F.CrtYd"))
-    (fp_line (start -1.6 0.95) (end 1.6 0.95)
-      (stroke (width 0.05) (type solid)) (layer "F.CrtYd"))
-    (fp_line (start 1.6 -0.95) (end 1.6 0.95)
-      (stroke (width 0.05) (type solid)) (layer "F.CrtYd"))
-    (fp_line (start -0.9 -0.7) (end 0.9 -0.7)
-      (stroke (width 0.1) (type solid)) (layer "F.Fab"))
-    (fp_line (start -0.9 0.7) (end -0.9 -0.7)
-      (stroke (width 0.1) (type solid)) (layer "F.Fab"))
-    (fp_line (start -0.3 -0.35) (end -0.3 0.35)
-      (stroke (width 0.1) (type solid)) (layer "F.Fab"))
-    (fp_line (start -0.3 0) (end -0.5 0)
-      (stroke (width 0.1) (type solid)) (layer "F.Fab"))
-    (fp_line (start -0.3 0) (end 0.2 -0.35)
-      (stroke (width 0.1) (type solid)) (layer "F.Fab"))
-    (fp_line (start 0.2 -0.35) (end 0.2 0.35)
-      (stroke (width 0.1) (type solid)) (layer "F.Fab"))
-    (fp_line (start 0.2 0) (end 0.45 0)
-      (stroke (width 0.1) (type solid)) (layer "F.Fab"))
-    (fp_line (start 0.2 0.35) (end -0.3 0)
-      (stroke (width 0.1) (type solid)) (layer "F.Fab"))
-    (fp_line (start 0.9 -0.7) (end 0.9 0.7)
-      (stroke (width 0.1) (type solid)) (layer "F.Fab"))
-    (fp_line (start 0.9 0.7) (end -0.9 0.7)
-      (stroke (width 0.1) (type solid)) (layer "F.Fab"))
-    (pad "1" smd roundrect (at -1.05 0 90) (size 0.6 0.45) (layers "F.Cu" "F.Paste" "F.Mask") (roundrect_rratio 0.25)
-      (net 111 "VCC") (pinfunction "K") (pintype "passive"))
-    (pad "2" smd roundrect (at 1.05 0 90) (size 0.6 0.45) (layers "F.Cu" "F.Paste" "F.Mask") (roundrect_rratio 0.25)
-      (net 112 "Net-(D1-A)") (pinfunction "A") (pintype "passive"))
-    (model "${KICAD6_3DMODEL_DIR}/Diode_SMD.3dshapes/D_SOD-323.wrl"
-      (offset (xyz 0 0 0))
-      (scale (xyz 1 1 1))
-      (rotate (xyz 0 0 0))
-    )
-  )
   (footprint "pkl_tag_connect:TC2030-NL_SMALL" (layer "F.Cu")
     (at 147.7264 47.625 180)
@@
     )
   )
+  (footprint "Diode_SMD:D_SOD-323" (layer "B.Cu")
+    (at 185.17 75.1775 90)
+    (descr "SOD-323")
+    (tags "SOD-323")
+    (property "Sheetfile" "pdclk.kicad_sch")
+    (property "Sheetname" "PD and CLK")
+    (property "ki_description" "10V 3A High Current Recitifier Schottky Diode, SOD-323")
+    (property "ki_keywords" "diode Schottky")
+    (attr smd)
+    (fp_text reference "D1" (at 0 -1.7312 90) (layer "B.SilkS")
+        (effects (font (size 1 1) (thickness 0.15)) (justify mirror))
+    )
+    (fp_text value "BAT60A" (at 0.1 -1.9 90) (layer "B.Fab") hide
+        (effects (font (size 1 1) (thickness 0.15)) (justify mirror))
+    )
+    (fp_text user "${REFERENCE}" (at 0 1.85 90) (layer "B.Fab")
+        (effects (font (size 1 1) (thickness 0.15)) (justify mirror))
+    )
+    (fp_line (start -1.61 -0.85) (end 1.05 -0.85)
+      (stroke (width 0.12) (type solid)) (layer "B.SilkS"))
+    (fp_line (start -1.61 0.85) (end -1.61 -0.85)
+      (stroke (width 0.12) (type solid)) (layer "B.SilkS"))
+    (fp_line (start -1.61 0.85) (end 1.05 0.85)
+      (stroke (width 0.12) (type solid)) (layer "B.SilkS"))
+    (fp_line (start -1.6 -0.95) (end 1.6 -0.95)
+      (stroke (width 0.05) (type solid)) (layer "B.CrtYd"))
+    (fp_line (start -1.6 0.95) (end -1.6 -0.95)
+      (stroke (width 0.05) (type solid)) (layer "B.CrtYd"))
+    (fp_line (start -1.6 0.95) (end 1.6 0.95)
+      (stroke (width 0.05) (type solid)) (layer "B.CrtYd"))
+    (fp_line (start 1.6 0.95) (end 1.6 -0.95)
+      (stroke (width 0.05) (type solid)) (layer "B.CrtYd"))
+    (fp_line (start -0.9 -0.7) (end -0.9 0.7)
+      (stroke (width 0.1) (type solid)) (layer "B.Fab"))
+    (fp_line (start -0.9 0.7) (end 0.9 0.7)
+      (stroke (width 0.1) (type solid)) (layer "B.Fab"))
+    (fp_line (start -0.3 0) (end -0.5 0)
+      (stroke (width 0.1) (type solid)) (layer "B.Fab"))
+    (fp_line (start -0.3 0) (end 0.2 0.35)
+      (stroke (width 0.1) (type solid)) (layer "B.Fab"))
+    (fp_line (start -0.3 0.35) (end -0.3 -0.35)
+      (stroke (width 0.1) (type solid)) (layer "B.Fab"))
+    (fp_line (start 0.2 -0.35) (end -0.3 0)
+      (stroke (width 0.1) (type solid)) (layer "B.Fab"))
+    (fp_line (start 0.2 0) (end 0.45 0)
+      (stroke (width 0.1) (type solid)) (layer "B.Fab"))
+    (fp_line (start 0.2 0.35) (end 0.2 -0.35)
+      (stroke (width 0.1) (type solid)) (layer "B.Fab"))
+    (fp_line (start 0.9 -0.7) (end -0.9 -0.7)
+      (stroke (width 0.1) (type solid)) (layer "B.Fab"))
+    (fp_line (start 0.9 0.7) (end 0.9 -0.7)
+      (stroke (width 0.1) (type solid)) (layer "B.Fab"))
+    (pad "1" smd roundrect (at -1.05 0 90) (size 0.6 0.45) (layers "B.Cu" "B.Paste" "B.Mask") (roundrect_rratio 0.25)
+      (net 111 "VCC") (pinfunction "K") (pintype "passive"))
+    (pad "2" smd roundrect (at 1.05 0 90) (size 0.6 0.45) (layers "B.Cu" "B.Paste" "B.Mask") (roundrect_rratio 0.25)
+      (net 112 "Net-(D1-A)") (pinfunction "A") (pintype "passive"))
+    (model "${KICAD6_3DMODEL_DIR}/Diode_SMD.3dshapes/D_SOD-323.wrl"
+      (offset (xyz 0 0 0))
+      (scale (xyz 1 1 1))
+      (rotate (xyz 0 0 0))
+    )
+  )
   (footprint "Package_DFN_QFN:QFN-20-1EP_3x3mm_P0.45mm_EP1.6x1.6mm" (layer "B.Cu")
     (at 102.1566 57.9518 180)
@@
   (segment (start 170.998 54.8184) (end 170.998 54.09) (width 0.25) (layer "B.Cu") (net 110))
   (segment (start 174.9806 58.801) (end 170.998 54.8184) (width 0.25) (layer "B.Cu") (net 110))
-  (segment (start 185.92 77.76) (end 189.85 77.76) (width 0.4) (layer "F.Cu") (net 111))
-  (segment (start 185.17 77.01) (end 185.92 77.76) (width 0.4) (layer "F.Cu") (net 111))
-  (segment (start 185.17 76.2275) (end 185.17 77.01) (width 0.4) (layer "F.Cu") (net 111))
-  (segment (start 189.85 77.76) (end 190.61 77) (width 0.4) (layer "F.Cu") (net 111))
-  (segment (start 190.61 77) (end 190.61 75.23) (width 0.4) (layer "F.Cu") (net 111))
-  (segment (start 187.34 72.82) (end 185.88 72.82) (width 0.4) (layer "F.Cu") (net 112))
-  (segment (start 185.88 72.82) (end 185.17 73.53) (width 0.4) (layer "F.Cu") (net 112))
-  (segment (start 188.07 73.55) (end 187.34 72.82) (width 0.4) (layer "F.Cu") (net 112))
-  (segment (start 188.07 75.23) (end 188.07 73.55) (width 0.4) (layer "F.Cu") (net 112))
-  (segment (start 185.17 73.53) (end 185.17 74.1275) (width 0.4) (layer "F.Cu") (net 112))
+  (segment (start 185.92 77.76) (end 189.85 77.76) (width 0.4) (layer "B.Cu") (net 111))
+  (segment (start 185.17 77.01) (end 185.92 77.76) (width 0.4) (layer "B.Cu") (net 111))
+  (segment (start 185.17 76.2275) (end 185.17 77.01) (width 0.4) (layer "B.Cu") (net 111))
+  (segment (start 189.85 77.76) (end 190.61 77) (width 0.4) (layer "B.Cu") (net 111))
+  (segment (start 190.61 77) (end 190.61 75.23) (width 0.4) (layer "B.Cu") (net 111))
+  (segment (start 187.34 72.82) (end 185.88 72.82) (width 0.4) (layer "B.Cu") (net 112))
+  (segment (start 185.88 72.82) (end 185.17 73.53) (width 0.4) (layer "B.Cu") (net 112))
+  (segment (start 188.07 73.55) (end 187.34 72.82) (width 0.4) (layer "B.Cu") (net 112))
+  (segment (start 188.07 75.23) (end 188.07 73.55) (width 0.4) (layer "B.Cu") (net 112))
+  (segment (start 185.17 73.53) (end 185.17 74.1275) (width 0.4) (layer "B.Cu") (net 112))
   (zone (net 2) (net_name "GND") (layer "In2.Cu") (hatch edge 0.5)
     (connect_pads (clearance 0.5))

Commit message: Added BOM csv and part numbers to PCB
Parts:
- D1: value BAT60A -> BAT60AE6327HTSA1
- U3, U9: value ATtiny44A-MMH -> ATTINY44A-MMHR
Changed lines of the file:
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@@
+        (effects (font (size 1 1) (thickness 0.15)))
+    )
+    (fp_text user "48-6554-11" (at 0 0 90 unlocked) (layer "F.Fab") hide
         (effects (font (size 1 1) (thickness 0.15)))
     )
@@
         (effects (font (size 1 1) (thickness 0.15)))
     )
+    (fp_text user "48-6554-11" (at 0 0 -90 unlocked) (layer "F.Fab") hide
+        (effects (font (size 1 1) (thickness 0.15)))
+    )
     (fp_line (start -1.33 -1.33) (end 0 -1.33)
       (stroke (width 0.12) (type solid)) (layer "F.SilkS"))
@@
         (effects (font (size 1 1) (thickness 0.15)))
     )
+    (fp_text user "1718561008" (at 0 0 180 unlocked) (layer "F.Fab") hide
+        (effects (font (size 1 1) (thickness 0.15)))
+    )
     (fp_line (start -1.33 -1.33) (end 0 -1.33)
       (stroke (width 0.12) (type solid)) (layer "F.SilkS"))
@@
     (fp_text user "${REFERENCE}" (at 0 0) (layer "B.Fab") hide
         (effects (font (size 0.4 0.4) (thickness 0.06)) (justify mirror))
+    )
+    (fp_text user "CC0603KPX7R7BB105" (at 0 0 unlocked) (layer "B.Fab") hide
+        (effects (font (size 1 1) (thickness 0.15)) (justify mirror))
     )
     (fp_line (start -0.146267 -0.51) (end 0.146267 -0.51)
@@
     (property "ki_keywords" "R res resistor")
     (attr smd)
-    (fp_text reference "R1" (at 2.4561 0.1524 -180) (layer "B.SilkS")
+    (fp_text reference "R1" (at 2.4561 0.1524) (layer "B.SilkS")
         (effects (font (size 1 1) (thickness 0.15)) (justify mirror))
     )
     (fp_text value "100R" (at 0 -1.43 90) (layer "B.Fab") hide
+        (effects (font (size 1 1) (thickness 0.15)) (justify mirror))
+    )
+    (fp_text user "RC0603FR-07100RL" (at 0 0 -90 unlocked) (layer "B.Fab") hide
         (effects (font (size 1 1) (thickness 0.15)) (justify mirror))
     )
@@
     (property "ki_keywords" "cap capacitor")
     (attr smd)
-    (fp_text reference "C1" (at -0.478 1.824 -180) (layer "B.SilkS")
+    (fp_text reference "C1" (at -0.478 1.824) (layer "B.SilkS")
         (effects (font (size 1 1) (thickness 0.15)) (justify mirror))
     )
     (fp_text value "1uF" (at 0 -1.43 -270) (layer "B.Fab") hide
+        (effects (font (size 1 1) (thickness 0.15)) (justify mirror))
+    )
+    (fp_text user "CC0603KPX7R7BB105" (at 0 0 -90 unlocked) (layer "B.Fab") hide
         (effects (font (size 1 1) (thickness 0.15)) (justify mirror))
     )
@@
         (effects (font (size 1 1) (thickness 0.15)) (justify mirror))
     )
-    (fp_text value "ATtiny44A-MMH" (at 0 -2.82) (layer "B.Fab") hide
+    (fp_text value "ATTINY44A-MMHR" (at 0 -2.82) (layer "B.Fab") hide
         (effects (font (size 1 1) (thickness 0.15)) (justify mirror))
     )
@@
         (effects (font (size 1 1) (thickness 0.15)) (justify mirror))
     )
-    (fp_text value "BAT60A" (at 0.1 -1.9 90) (layer "B.Fab") hide
+    (fp_text value "BAT60AE6327HTSA1" (at 0.1 -1.9 90) (layer "B.Fab") hide
         (effects (font (size 1 1) (thickness 0.15)) (justify mirror))
     )
@@
         (effects (font (size 1 1) (thickness 0.15)) (justify mirror))
     )
-    (fp_text value "ATtiny44A-MMH" (at 0 -2.82) (layer "B.Fab") hide
+    (fp_text value "ATTINY44A-MMHR" (at 0 -2.82) (layer "B.Fab") hide
         (effects (font (size 1 1) (thickness 0.15)) (justify mirror))
     )
@@
         (effects (font (size 0.4 0.4) (thickness 0.06)) (justify mirror))
     )
+    (fp_text user "RC0603FR-0710KL" (at 0 0 90 unlocked) (layer "B.Fab") hide
+        (effects (font (size 1 1) (thickness 0.15)) (justify mirror))
+    )
     (fp_line (start -0.254724 -0.5225) (end 0.254724 -0.5225)
       (stroke (width 0.12) (type solid)) (layer "B.SilkS"))
@@
     (property "ki_keywords" "cap capacitor")
     (attr smd)
-    (fp_text reference "C3" (at -2.2595 0 -180) (layer "B.SilkS")
+    (fp_text reference "C3" (at -2.2595 0) (layer "B.SilkS")
         (effects (font (size 1 1) (thickness 0.15)) (justify mirror))
     )
@@
     (fp_text user "${REFERENCE}" (at 0 0 90) (layer "B.Fab") hide
         (effects (font (size 0.4 0.4) (thickness 0.06)) (justify mirror))
+    )
+    (fp_text user "CC0603KPX7R7BB105" (at 0 0 -90 unlocked) (layer "B.Fab") hide
+        (effects (font (size 1 1) (thickness 0.15)) (justify mirror))
     )
     (fp_line (start -0.146267 -0.51) (end 0.146267 -0.51)
@@
     (property "ki_keywords" "cap capacitor")
     (attr smd)
-    (fp_text reference "C4" (at -0.1259 -1.7272 -180) (layer "B.SilkS")
+    (fp_text reference "C4" (at -0.1259 -1.7272) (layer "B.SilkS")
         (effects (font (size 1 1) (thickness 0.15)) (justify mirror))
     )
@@
     (fp_text user "${REFERENCE}" (at 0 0 90) (layer "B.Fab") hide
         (effects (font (size 0.4 0.4) (thickness 0.06)) (justify mirror))
+    )
+    (fp_text user "CC0603KRX7RBB104" (at 0 0 -90 unlocked) (layer "B.Fab") hide
+        (effects (font (size 1 1) (thickness 0.15)) (justify mirror))
     )
     (fp_line (start -0.146267 -0.51) (end 0.146267 -0.51)
@@
     (property "ki_keywords" "cap capacitor")
     (attr smd)
-    (fp_text reference "C6" (at -2.286 -0.0254 -180) (layer "B.SilkS")
+    (fp_text reference "C6" (at -2.286 -0.0254) (layer "B.SilkS")
         (effects (font (size 1 1) (thickness 0.15)) (justify mirror))
     )
     (fp_text value "1uF" (at 0 -1.43 90) (layer "B.Fab") hide
+        (effects (font (size 1 1) (thickness 0.15)) (justify mirror))
+    )
+    (fp_text user "CC0603KPX7R7BB105" (at 0 0 -90 unlocked) (layer "B.Fab") hide
         (effects (font (size 1 1) (thickness 0.15)) (justify mirror))
     )
@@
         (effects (font (size 0.4 0.4) (thickness 0.06)) (justify mirror))
     )
+    (fp_text user "CC0603KRX7RBB104" (at 0 0 180 unlocked) (layer "B.Fab") hide
+        (effects (font (size 1 1) (thickness 0.15)) (justify mirror))
+    )
     (fp_line (start -0.146267 -0.51) (end 0.146267 -0.51)
       (stroke (width 0.12) (type solid)) (layer "B.SilkS"))
@@
     (property "ki_keywords" "R res resistor")
     (attr smd)
-    (fp_text reference "R3" (at 2.4384 0.0254 -180) (layer "B.SilkS")
+    (fp_text reference "R3" (at 2.4384 0.0254) (layer "B.SilkS")
         (effects (font (size 1 1) (thickness 0.15)) (justify mirror))
     )
@@
     (fp_text user "${REFERENCE}" (at 0 0 90) (layer "B.Fab") hide
         (effects (font (size 0.4 0.4) (thickness 0.06)) (justify mirror))
+    )
+    (fp_text user "RC0603FR-07100RL" (at 0 0 -90 unlocked) (layer "B.Fab") hide
+        (effects (font (size 1 1) (thickness 0.15)) (justify mirror))
     )
     (fp_line (start -0.254724 -0.5225) (end 0.254724 -0.5225)
@@
         (effects (font (size 1 1) (thickness 0.15)) (justify mirror))
     )
+    (fp_text user "RC0603FR-0710KL" (at 0 0 90 unlocked) (layer "B.Fab") hide
+        (effects (font (size 1 1) (thickness 0.15)) (justify mirror))
+    )
     (fp_text user "${REFERENCE}" (at 0 0 90) (layer "B.Fab") hide
         (effects (font (size 0.4 0.4) (thickness 0.06)) (justify mirror))
@@
         (effects (font (size 0.4 0.4) (thickness 0.06)) (justify mirror))
     )
+    (fp_text user "CC0603KRX7RBB104" (at 0 0 180 unlocked) (layer "B.Fab") hide
+        (effects (font (size 1 1) (thickness 0.15)) (justify mirror))
+    )
     (fp_line (start -0.146267 -0.51) (end 0.146267 -0.51)
       (stroke (width 0.12) (type solid)) (layer "B.SilkS"))
@@
     (property "ki_keywords" "cap capacitor")
     (attr smd)
-    (fp_text reference "C7" (at 0.0519 -1.778 -180) (layer "B.SilkS")
+    (fp_text reference "C7" (at 0.0519 -1.778) (layer "B.SilkS")
         (effects (font (size 1 1) (thickness 0.15)) (justify mirror))
     )
@@
         (effects (font (size 1 1) (thickness 0.15)) (justify mirror))
     )
+    (fp_text user "CC0603KRX7RBB104" (at 0 0 -90 unlocked) (layer "B.Fab") hide
+        (effects (font (size 1 1) (thickness 0.15)) (justify mirror))
+    )
